File: main-oscillator.sch (EAGLE design)
At the start: 15 parts, among them IC1 7805TV, IC2 UA555N

Commit message: Smaller transformer, DIL package for rectifier bridge. More compact design.
Parts:
- removed C2: 470n, rcl:C-EU050-030X075
- removed X1: (no value), con-wago-500:W237-103
- added JP1: mains, SparkFun-Connectors:M03-SCREW-5MM
- B1: device rectifier:RECTIFIER-KBL -> rectifier:B-DIL
- R1: value 1k -> 100R
- R3: value 330k -> 220k
- TR1: value 230-9V -> 230-6V; device trafo:EI30-2 -> trafo:EE20-2
Connections:
- net GND: no longer C2.2
- net N$1: now also JP1.3; no longer X1-3.KL
- net N$2: now also TR1.3; no longer TR1.4
- net N$3: now also JP1.1; no longer X1-1.KL
- net N$4: now also JP1.2; no longer X1-2.KL
- net N$5: no longer C2.1
- net N$6: now also TR1.4; no longer TR1.3
Changed lines of the file:
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@@
 <setting verticaltext="up"/>
 </settings>
-<grid distance="0.1" unitdist="inch" unit="inch" style="lines" multiple="1" display="yes" altdistance="0.01" altunitdist="inch" altunit="inch"/>
+<grid distance="0.1" unitdist="inch" unit="inch" style="lines" multiple="1" display="no" altdistance="0.01" altunitdist="inch" altunit="inch"/>
 <layers>
 <layer number="1" name="Top" color="4" fill="1" visible="no" active="no"/>
@@
 </classes>
 <parts>
-<part name="TR1" library="trafo" deviceset="EI30-2" device="" value="230-9V"/>
-<part name="C2" library="rcl" deviceset="C-EU" device="050-030X075" value="470n"/>
+<part name="TR1" library="trafo" deviceset="EE20-2" device="" value="230-6V"/>
 <part name="R2" library="resistor" deviceset="R-EU_" device="0207/10" value="1k"/>
-<part name="B1" library="rectifier" deviceset="RECTIFIER-" device="KBL" value="RECTIFIER-KBL"/>
+<part name="B1" library="rectifier" deviceset="B-DIL" device="" value="RECTIFIER-KBL"/>
 <part name="IC2" library="linear" deviceset="*555" device="N" technology="UA"/>
 <part name="IC1" library="linear" deviceset="78*" device="TV" technology="05"/>
 <part name="C3" library="resistor" deviceset="C-EU" device="050-024X044" value="100n"/>
-<part name="R1" library="resistor" deviceset="R-EU_" device="0207/10" value="1k"/>
+<part name="R1" library="resistor" deviceset="R-EU_" device="0207/10" value="100R"/>
 <part name="C5" library="rcl" deviceset="C-EU" device="025-025X050" value="10n"/>
 <part name="C4" library="rcl" deviceset="CPOL-EU" device="E5-13" value="32u"/>
@@
 <part name="C6" library="resistor" deviceset="C-EU" device="050-024X044" value="100n"/>
 <part name="BNC11" library="SparkFun-Connectors" deviceset="BNC" device="PTH"/>
-<part name="R3" library="resistor" deviceset="R-EU_" device="0207/10" value="330k"/>
-<part name="X1" library="con-wago-500" deviceset="W237-103" device=""/>
+<part name="R3" library="resistor" deviceset="R-EU_" device="0207/10" value="220k"/>
+<part name="JP1" library="SparkFun-Connectors" deviceset="M03" device="-SCREW-5MM" value="mains"/>
 </parts>
 <sheets>
@@
 <instances>
 <instance part="TR1" gate="1" x="12.7" y="25.4"/>
-<instance part="C2" gate="G$1" x="68.58" y="25.4"/>
 <instance part="R2" gate="G$1" x="119.38" y="20.32" rot="R90"/>
-<instance part="B1" gate="G$1" x="45.72" y="22.86" rot="MR0"/>
+<instance part="B1" gate="1" x="45.72" y="22.86" rot="MR0"/>
 <instance part="IC2" gate="A" x="149.86" y="22.86"/>
 <instance part="IC1" gate="A1" x="81.28" y="27.94"/>
@@
 <instance part="BNC11" gate="G$1" x="180.34" y="25.4" rot="MR0"/>
 <instance part="R3" gate="G$1" x="7.62" y="5.08" rot="R180"/>
-<instance part="X1" gate="-1" x="-7.62" y="17.78"/>
-<instance part="X1" gate="-2" x="-7.62" y="25.4"/>
-<instance part="X1" gate="-3" x="-7.62" y="30.48"/>
+<instance part="JP1" gate="G$1" x="-10.16" y="25.4"/>
 </instances>
 <busses>
@@
 <net name="GND" class="0">
 <segment>
-<pinref part="B1" gate="G$1" pin="-"/>
+<pinref part="B1" gate="1" pin="-"/>
 <wire x1="50.8" y1="22.86" x2="58.42" y2="22.86" width="0.1524" layer="91"/>
 <wire x1="58.42" y1="22.86" x2="58.42" y2="20.32" width="0.1524" layer="91"/>
 <pinref part="C3" gate="G$1" pin="2"/>
 <wire x1="58.42" y1="20.32" x2="60.96" y2="20.32" width="0.1524" layer="91"/>
-<pinref part="C2" gate="G$1" pin="2"/>
-<junction x="68.58" y="20.32"/>
-<wire x1="60.96" y1="20.32" x2="68.58" y2="20.32" width="0.1524" layer="91"/>
-<wire x1="68.58" y1="20.32" x2="81.28" y2="20.32" width="0.1524" layer="91"/>
+<wire x1="60.96" y1="20.32" x2="81.28" y2="20.32" width="0.1524" layer="91"/>
 <pinref part="IC1" gate="A1" pin="GND"/>
 <junction x="81.28" y="20.32"/>
@@
 <net name="N$5" class="0">
 <segment>
-<pinref part="B1" gate="G$1" pin="+"/>
+<pinref part="B1" gate="1" pin="+"/>
 <wire x1="40.64" y1="22.86" x2="35.56" y2="22.86" width="0.1524" layer="91"/>
 <wire x1="35.56" y1="22.86" x2="35.56" y2="38.1" width="0.1524" layer="91"/>
@@
 <wire x1="35.56" y1="38.1" x2="60.96" y2="38.1" width="0.1524" layer="91"/>
 <wire x1="60.96" y1="38.1" x2="60.96" y2="27.94" width="0.1524" layer="91"/>
-<pinref part="C2" gate="G$1" pin="1"/>
 <pinref part="IC1" gate="A1" pin="VI"/>
-<wire x1="71.12" y1="27.94" x2="68.58" y2="27.94" width="0.1524" layer="91"/>
-<wire x1="60.96" y1="27.94" x2="68.58" y2="27.94" width="0.1524" layer="91"/>
+<wire x1="60.96" y1="27.94" x2="71.12" y2="27.94" width="0.1524" layer="91"/>
 <junction x="60.96" y="27.94"/>
-<junction x="68.58" y="27.94"/>
 </segment>
 </net>
@@
 <pinref part="R1" gate="G$1" pin="2"/>
 <wire x1="96.52" y1="40.64" x2="119.38" y2="40.64" width="0.1524" layer="91"/>
-<pinref part="IC2" gate="A" pin="V+"/>
-<wire x1="165.1" y1="22.86" x2="160.02" y2="15.24" width="0.1524" layer="91"/>
 <pinref part="IC2" gate="A" pin="R"/>
-<wire x1="139.7" y1="25.4" x2="165.1" y2="22.86" width="0.1524" layer="91"/>
-<junction x="139.7" y="25.4"/>
 <wire x1="137.16" y1="25.4" x2="139.7" y2="25.4" width="0.1524" layer="91"/>
 <wire x1="119.38" y1="40.64" x2="137.16" y2="40.64" width="0.1524" layer="91"/>
@@
 <junction x="119.38" y="40.64"/>
 <label x="111.76" y="43.18" size="1.778" layer="95"/>
+<pinref part="IC2" gate="A" pin="V+"/>
+<wire x1="165.1" y1="22.86" x2="160.02" y2="15.24" width="0.1524" layer="91"/>
 <pinref part="C6" gate="G$1" pin="1"/>
 <junction x="160.02" y="15.24"/>
+<wire x1="165.1" y1="22.86" x2="165.1" y2="27.94" width="0.1524" layer="91"/>
+<wire x1="165.1" y1="27.94" x2="144.78" y2="27.94" width="0.1524" layer="91"/>
+<wire x1="144.78" y1="27.94" x2="144.78" y2="25.4" width="0.1524" layer="91"/>
+<wire x1="144.78" y1="25.4" x2="139.7" y2="25.4" width="0.1524" layer="91"/>
+<junction x="139.7" y="25.4"/>
 </segment>
 </net>
@@
 <net name="N$2" class="0">
 <segment>
-<pinref part="TR1" gate="1" pin="4"/>
-<wire x1="20.32" y1="22.86" x2="30.48" y2="22.86" width="0.1524" layer="91"/>
-<wire x1="30.48" y1="22.86" x2="30.48" y2="17.78" width="0.1524" layer="91"/>
-<pinref part="B1" gate="G$1" pin="AC2"/>
-<wire x1="30.48" y1="17.78" x2="45.72" y2="17.78" width="0.1524" layer="91"/>
+<pinref part="B1" gate="1" pin="AC2"/>
+<wire x1="20.32" y1="17.78" x2="45.72" y2="17.78" width="0.1524" layer="91"/>
 <wire x1="45.72" y1="17.78" x2="53.34" y2="17.78" width="0.1524" layer="91"/>
 <junction x="45.72" y="17.78"/>
@@
 <wire x1="104.14" y1="30.48" x2="104.14" y2="45.72" width="0.1524" layer="91"/>
 <wire x1="53.34" y1="17.78" x2="53.34" y2="45.72" width="0.1524" layer="91"/>
-</segment>
-</net>
-<net name="N$6" class="0">
-<segment>
 <pinref part="TR1" gate="1" pin="3"/>
-<wire x1="20.32" y1="17.78" x2="25.4" y2="17.78" width="0.1524" layer="91"/>
-<wire x1="25.4" y1="17.78" x2="25.4" y2="27.94" width="0.1524" layer="91"/>
-<pinref part="B1" gate="G$1" pin="AC1"/>
-<wire x1="25.4" y1="27.94" x2="45.72" y2="27.94" width="0.1524" layer="91"/>
 </segment>
 </net>
 <net name="N$4" class="0">
 <segment>
-<pinref part="X1" gate="-2" pin="KL"/>
 <pinref part="R3" gate="G$1" pin="2"/>
+<wire x1="2.54" y1="25.4" x2="2.54" y2="5.08" width="0.1524" layer="91"/>
+<pinref part="JP1" gate="G$1" pin="2"/>
 <wire x1="-2.54" y1="25.4" x2="2.54" y2="25.4" width="0.1524" layer="91"/>
-<wire x1="2.54" y1="25.4" x2="2.54" y2="5.08" width="0.1524" layer="91"/>
 </segment>
 </net>
 <net name="N$1" class="0">
 <segment>
-<pinref part="X1" gate="-3" pin="KL"/>
 <pinref part="TR1" gate="1" pin="1"/>
 <wire x1="-2.54" y1="30.48" x2="7.62" y2="30.48" width="0.1524" layer="91"/>
+<pinref part="JP1" gate="G$1" pin="3"/>
+<wire x1="-2.54" y1="30.48" x2="-2.54" y2="27.94" width="0.1524" layer="91"/>
 </segment>
 </net>
@@
 <segment>
 <pinref part="TR1" gate="1" pin="2"/>
-<pinref part="X1" gate="-1" pin="KL"/>
 <wire x1="7.62" y1="17.78" x2="-2.54" y2="17.78" width="0.1524" layer="91"/>
-</segment>
-</net>
+<pinref part="JP1" gate="G$1" pin="1"/>
+<wire x1="-2.54" y1="22.86" x2="-2.54" y2="17.78" width="0.1524" layer="91"/>
+</segment>
+</net>
+<net name="N$6" class="0">
+<segment>
+<pinref part="B1" gate="1" pin="AC1"/>
+<wire x1="45.72" y1="27.94" x2="25.4" y2="27.94" width="0.1524" layer="91"/>
+<wire x1="25.4" y1="27.94" x2="25.4" y2="22.86" width="0.1524" layer="91"/>
+<pinref part="TR1" gate="1" pin="4"/>
+<wire x1="25.4" y1="22.86" x2="20.32" y2="22.86" width="0.1524" layer="91"/>
+</segment>
+</net>

Commit message: v 1.1: added switch gitignore updated with 'stuff' folder
Parts:
- added S1: (no value), switch:320-916
Connections:
- new net N$10: JP1.3, S1.S
- net N$1: now also S1.P; no longer JP1.3
- net N$2: now also TR1.5; no longer TR1.3
- net N$6: now also TR1.6; no longer TR1.4
Other:
- moved on the sheet: JP1, R3
Changed lines of the file:
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@@
 <grid distance="0.1" unitdist="inch" unit="inch" style="lines" multiple="1" display="no" altdistance="0.01" altunitdist="inch" altunit="inch"/>
 <layers>
-<layer number="1" name="Top" color="4" fill="1" visible="no" active="no"/>
-<layer number="16" name="Bottom" color="1" fill="1" visible="no" active="no"/>
-<layer number="17" name="Pads" color="2" fill="1" visible="no" active="no"/>
-<layer number="18" name="Vias" color="2" fill="1" visible="no" active="no"/>
-<layer number="19" name="Unrouted" color="6" fill="1" visible="no" active="no"/>
-<layer number="20" name="Dimension" color="15" fill="1" visible="no" active="no"/>
-<layer number="21" name="tPlace" color="7" fill="1" visible="no" active="no"/>
-<layer number="22" name="bPlace" color="7" fill="1" visible="no" active="no"/>
-<layer number="23" name="tOrigins" color="15" fill="1" visible="no" active="no"/>
-<layer number="24" name="bOrigins" color="15" fill="1" visible="no" active="no"/>
-<layer number="25" name="tNames" color="7" fill="1" visible="no" active="no"/>
-<layer number="26" name="bNames" color="7" fill="1" visible="no" active="no"/>
-<layer number="27" name="tValues" color="7" fill="1" visible="no" active="no"/>
-<layer number="28" name="bValues" color="7" fill="1" visible="no" active="no"/>
+<layer number="1" name="Top" color="4" fill="1" visible="yes" active="no"/>
+<layer number="16" name="Bottom" color="1" fill="1" visible="yes" active="no"/>
+<layer number="17" name="Pads" color="2" fill="1" visible="yes" active="no"/>
+<layer number="18" name="Vias" color="2" fill="1" visible="yes" active="no"/>
+<layer number="19" name="Unrouted" color="6" fill="1" visible="yes" active="no"/>
+<layer number="20" name="Dimension" color="15" fill="1" visible="yes" active="no"/>
+<layer number="21" name="tPlace" color="7" fill="1" visible="yes" active="no"/>
+<layer number="22" name="bPlace" color="7" fill="1" visible="yes" active="no"/>
+<layer number="23" name="tOrigins" color="15" fill="1" visible="yes" active="no"/>
+<layer number="24" name="bOrigins" color="15" fill="1" visible="yes" active="no"/>
+<layer number="25" name="tNames" color="7" fill="1" visible="yes" active="no"/>
+<layer number="26" name="bNames" color="7" fill="1" visible="yes" active="no"/>
+<layer number="27" name="tValues" color="7" fill="1" visible="yes" active="no"/>
+<layer number="28" name="bValues" color="7" fill="1" visible="yes" active="no"/>
 <layer number="29" name="tStop" color="7" fill="3" visible="no" active="no"/>
 <layer number="30" name="bStop" color="7" fill="6" visible="no" active="no"/>
@@
 <layer number="35" name="tGlue" color="7" fill="4" visible="no" active="no"/>
 <layer number="36" name="bGlue" color="7" fill="5" visible="no" active="no"/>
-<layer number="37" name="tTest" color="7" fill="1" visible="no" active="no"/>
-<layer number="38" name="bTest" color="7" fill="1" visible="no" active="no"/>
+<layer number="37" name="tTest" color="7" fill="1" visible="yes" active="no"/>
+<layer number="38" name="bTest" color="7" fill="1" visible="yes" active="no"/>
 <layer number="39" name="tKeepout" color="4" fill="11" visible="no" active="no"/>
 <layer number="40" name="bKeepout" color="1" fill="11" visible="no" active="no"/>
@@
 <layer number="44" name="Drills" color="7" fill="1" visible="no" active="no"/>
 <layer number="45" name="Holes" color="7" fill="1" visible="no" active="no"/>
-<layer number="46" name="Milling" color="3" fill="1" visible="no" active="no"/>
-<layer number="47" name="Measures" color="7" fill="1" visible="no" active="no"/>
-<layer number="48" name="Document" color="7" fill="1" visible="no" active="no"/>
-<layer number="49" name="Reference" color="7" fill="1" visible="no" active="no"/>
-<layer number="50" name="dxf" color="7" fill="1" visible="no" active="no"/>
-<layer number="51" name="tDocu" color="7" fill="1" visible="no" active="no"/>
-<layer number="52" name="bDocu" color="7" fill="1" visible="no" active="no"/>
-<layer number="53" name="tGND_GNDA" color="7" fill="9" visible="no" active="no"/>
-<layer number="54" name="bGND_GNDA" color="1" fill="9" visible="no" active="no"/>
-<layer number="56" name="wert" color="7" fill="1" visible="no" active="no"/>
-<layer number="57" name="tCAD" color="7" fill="1" visible="no" active="no"/>
+<layer number="46" name="Milling" color="3" fill="1" visible="yes" active="no"/>
+<layer number="47" name="Measures" color="7" fill="1" visible="yes" active="no"/>
+<layer number="48" name="Document" color="7" fill="1" visible="yes" active="no"/>
+<layer number="49" name="Reference" color="7" fill="1" visible="yes" active="no"/>
+<layer number="50" name="dxf" color="7" fill="1" visible="yes" active="no"/>
+<layer number="51" name="tDocu" color="7" fill="1" visible="yes" active="no"/>
+<layer number="52" name="bDocu" color="7" fill="1" visible="yes" active="no"/>
+<layer number="53" name="tGND_GNDA" color="7" fill="9" visible="yes" active="no"/>
+<layer number="54" name="bGND_GNDA" color="1" fill="9" visible="yes" active="no"/>
+<layer number="56" name="wert" color="7" fill="1" visible="yes" active="no"/>
+<layer number="57" name="tCAD" color="7" fill="1" visible="yes" active="no"/>
 <layer number="90" name="Modules" color="5" fill="1" visible="yes" active="yes"/>
 <layer number="91" name="Nets" color="2" fill="1" visible="yes" active="yes"/>
@@
 <part name="R3" library="resistor" deviceset="R-EU_" device="0207/10" value="220k"/>
 <part name="JP1" library="SparkFun-Connectors" deviceset="M03" device="-SCREW-5MM" value="mains"/>
+<part name="S1" library="switch" deviceset="320-916" device=""/>
 </parts>
 <sheets>
 <sheet>
+<description>50 Hz oscillator
+Lock the experiment to the mains</description>
 <plain>
 </plain>
@@
 <instance part="C6" gate="G$1" x="160.02" y="12.7"/>
 <instance part="BNC11" gate="G$1" x="180.34" y="25.4" rot="MR0"/>
-<instance part="R3" gate="G$1" x="7.62" y="5.08" rot="R180"/>
-<instance part="JP1" gate="G$1" x="-10.16" y="25.4"/>
+<instance part="R3" gate="G$1" x="5.08" y="5.08" rot="R180"/>
+<instance part="JP1" gate="G$1" x="-12.7" y="25.4"/>
+<instance part="S1" gate="1" x="0" y="35.56" rot="MR270"/>
 </instances>
 <busses>
@@
 <pinref part="C6" gate="G$1" pin="2"/>
 <junction x="160.02" y="7.62"/>
-<wire x1="12.7" y1="5.08" x2="60.96" y2="5.08" width="0.1524" layer="91"/>
+<wire x1="10.16" y1="5.08" x2="60.96" y2="5.08" width="0.1524" layer="91"/>
 <wire x1="60.96" y1="5.08" x2="60.96" y2="20.32" width="0.1524" layer="91"/>
 <pinref part="BNC11" gate="G$1" pin="GND"/>
@@
 <segment>
 <pinref part="B1" gate="1" pin="AC2"/>
-<wire x1="20.32" y1="17.78" x2="45.72" y2="17.78" width="0.1524" layer="91"/>
 <wire x1="45.72" y1="17.78" x2="53.34" y2="17.78" width="0.1524" layer="91"/>
-<junction x="45.72" y="17.78"/>
 <pinref part="C4" gate="G$1" pin="+"/>
 <wire x1="53.34" y1="45.72" x2="104.14" y2="45.72" width="0.1524" layer="91"/>
@@
 <wire x1="104.14" y1="30.48" x2="104.14" y2="45.72" width="0.1524" layer="91"/>
 <wire x1="53.34" y1="17.78" x2="53.34" y2="45.72" width="0.1524" layer="91"/>
-<pinref part="TR1" gate="1" pin="3"/>
+<pinref part="TR1" gate="1" pin="5"/>
+<wire x1="20.32" y1="25.4" x2="30.48" y2="25.4" width="0.1524" layer="91"/>
+<wire x1="30.48" y1="25.4" x2="30.48" y2="17.78" width="0.1524" layer="91"/>
+<wire x1="30.48" y1="17.78" x2="45.72" y2="17.78" width="0.1524" layer="91"/>
+<junction x="45.72" y="17.78"/>
 </segment>
 </net>
@@
 <segment>
 <pinref part="R3" gate="G$1" pin="2"/>
-<wire x1="2.54" y1="25.4" x2="2.54" y2="5.08" width="0.1524" layer="91"/>
+<wire x1="0" y1="25.4" x2="0" y2="5.08" width="0.1524" layer="91"/>
 <pinref part="JP1" gate="G$1" pin="2"/>
-<wire x1="-2.54" y1="25.4" x2="2.54" y2="25.4" width="0.1524" layer="91"/>
-</segment>
-</net>
-<net name="N$1" class="0">
-<segment>
-<pinref part="TR1" gate="1" pin="1"/>
-<wire x1="-2.54" y1="30.48" x2="7.62" y2="30.48" width="0.1524" layer="91"/>
-<pinref part="JP1" gate="G$1" pin="3"/>
-<wire x1="-2.54" y1="30.48" x2="-2.54" y2="27.94" width="0.1524" layer="91"/>
+<wire x1="-5.08" y1="25.4" x2="0" y2="25.4" width="0.1524" layer="91"/>
 </segment>
 </net>
@@
 <segment>
 <pinref part="TR1" gate="1" pin="2"/>
-<wire x1="7.62" y1="17.78" x2="-2.54" y2="17.78" width="0.1524" layer="91"/>
+<wire x1="7.62" y1="17.78" x2="-5.08" y2="17.78" width="0.1524" layer="91"/>
 <pinref part="JP1" gate="G$1" pin="1"/>
-<wire x1="-2.54" y1="22.86" x2="-2.54" y2="17.78" width="0.1524" layer="91"/>
+<wire x1="-5.08" y1="22.86" x2="-5.08" y2="17.78" width="0.1524" layer="91"/>
 </segment>
 </net>
@@
 <pinref part="B1" gate="1" pin="AC1"/>
 <wire x1="45.72" y1="27.94" x2="25.4" y2="27.94" width="0.1524" layer="91"/>
-<wire x1="25.4" y1="27.94" x2="25.4" y2="22.86" width="0.1524" layer="91"/>
-<pinref part="TR1" gate="1" pin="4"/>
-<wire x1="25.4" y1="22.86" x2="20.32" y2="22.86" width="0.1524" layer="91"/>
-</segment>
-</net>
+<wire x1="25.4" y1="27.94" x2="25.4" y2="30.48" width="0.1524" layer="91"/>
+<pinref part="TR1" gate="1" pin="6"/>
+<wire x1="25.4" y1="30.48" x2="20.32" y2="30.48" width="0.1524" layer="91"/>
+</segment>
+</net>
+<net name="N$1" class="0">
+<segment>
+<pinref part="S1" gate="1" pin="P"/>
+<pinref part="TR1" gate="1" pin="1"/>
+<wire x1="5.08" y1="33.02" x2="7.62" y2="33.02" width="0.1524" layer="91"/>
+<wire x1="7.62" y1="33.02" x2="7.62" y2="30.48" width="0.1524" layer="91"/>
+</segment>
+</net>
+<net name="N$10" class="0">
+<segment>
+<pinref part="S1" gate="1" pin="S"/>
+<pinref part="JP1" gate="G$1" pin="3"/>
+<wire x1="-5.08" y1="30.48" x2="-5.08" y2="27.94" width="0.1524" layer="91"/>
+</segment>
+</net>
